Commit message: Description ROS 2 port

File: ridgeback_description/urdf/ridgeback.urdf.xacro (robot description, xacro)
@@ -63,227 +63,228 @@
     </transmission>
   </xacro:macro>
-  <xacro:macro name="rocker" params="prefix joint_type location *joint_limits">
-    <link name="${prefix}_rocker_link">
-      <visual>
-        <origin xyz="0 0 0" rpy="${PI/2} 0 ${PI/2}" />
-        <geometry>
-          <mesh filename="package://ridgeback_description/meshes/rocker.stl"/>
-        </geometry>
-        <material name="black" />
-      </visual>
+  <xacro:macro name="ridgeback">
+    <xacro:macro name="rocker" params="prefix joint_type location *joint_limits">
+      <link name="${prefix}_rocker_link">
+        <visual>
+          <origin xyz="0 0 0" rpy="${PI/2} 0 ${PI/2}" />
+          <geometry>
+            <mesh filename="package://ridgeback_description/meshes/rocker.stl"/>
+          </geometry>
+          <material name="black" />
+        </visual>
+        <inertial>
+          <origin xyz="0 0 0" rpy="${PI/2} 0 ${PI/2}"/>
+          <mass value="10.267"/>
+          <inertia
+            ixx="0.0288" ixy="2.20484e-6" ixz="-1.3145e-5"
+            iyy="0.4324" iyz="1.8944e-3"
+            izz="0.4130"/>
+        </inertial>
+      </link>
+      <joint name="${prefix}_rocker" type="${joint_type}">
+        <parent link="axle_link"/>
+        <child link="${prefix}_rocker_link" />
+        <origin xyz="${location*rocker_offset} 0 0" rpy="0 0 0" />
+        <axis xyz="1 0 0" />
+        <xacro:insert_block name="joint_limits" />
+      </joint>
+      <xacro:wheel prefix="${prefix}" side="left">
+        <origin xyz="0 ${rocker_width/2 + wheel_width/2} 0" rpy="0 0 0" />
+      </xacro:wheel>
+      <xacro:wheel prefix="${prefix}" side="right">
+        <origin xyz="0 ${-(rocker_width/2 + wheel_width/2)} 0" rpy="0 0 0" />
+      </xacro:wheel>
+    </xacro:macro>
+    <xacro:rocker prefix="front" joint_type="revolute" location="1" >
+      <limit lower="-0.08726" upper="0.08726" effort="0" velocity="0" />
+    </xacro:rocker>
+    <xacro:rocker prefix="rear" joint_type="fixed" location="-1" >
+      <limit effort="0" velocity="0" />
+    </xacro:rocker>
+    <joint name="base_link_joint" type="fixed">
+      <origin xyz="0 0 0" rpy="0 0 0" />
+      <parent link="base_link"/>
+      <child link="chassis_link" />
+    </joint>
+    <link name="chassis_link">
+      <visual>
+        <origin xyz="0 0 0" rpy="0 0 0" />
+        <geometry>
+          <mesh filename="package://ridgeback_description/meshes/body.stl"/>
+        </geometry>
+        <material name="black" />
+      </visual>
+      <collision>
+        <origin xyz="0 0 0"/>
+        <geometry>
+          <mesh filename="package://ridgeback_description/meshes/body-collision.stl"/>
+        </geometry>
+      </collision>
       <inertial>
-        <origin xyz="0 0 0" rpy="${PI/2} 0 ${PI/2}"/>
-        <mass value="10.267"/>
+        <origin xyz="0.012 0.002 0.067" rpy="${PI/2} 0 ${PI/2}"/>
+        <mass value="165.304"/>
         <inertia
-          ixx="0.0288" ixy="2.20484e-6" ixz="-1.3145e-5"
-          iyy="0.4324" iyz="1.8944e-3"
-          izz="0.4130"/>
+          ixx="4.4744" ixy="0.03098" ixz="0.003647"
+          iyy="7.1624" iyz="0.1228"
+          izz="4.6155"/>
       </inertial>
     </link>
-    <joint name="${prefix}_rocker" type="${joint_type}">
-      <parent link="axle_link"/>
-      <child link="${prefix}_rocker_link" />
-      <origin xyz="${location*rocker_offset} 0 0" rpy="0 0 0" />
-      <axis xyz="1 0 0" />
-      <xacro:insert_block name="joint_limits" />
-    </joint>
-    <xacro:wheel prefix="${prefix}" side="left">
-      <origin xyz="0 ${rocker_width/2 + wheel_width/2} 0" rpy="0 0 0" />
-    </xacro:wheel>
-    <xacro:wheel prefix="${prefix}" side="right">
-      <origin xyz="0 ${-(rocker_width/2 + wheel_width/2)} 0" rpy="0 0 0" />
-    </xacro:wheel>
+    <link name="riser_link">
+      <visual>
+        <origin xyz="0 0 ${riser_height/2}" rpy="0 0 ${pi/4}" />
+        <geometry>
+          <box size="0.493 0.493 ${riser_height}" />
+        </geometry>
+        <material name="light_grey" />
+      </visual>
+      <collision>
+        <origin xyz="0 0 ${riser_height/2}" rpy="0 0 ${pi/4}" />
+        <geometry>
+          <box size="0.493 0.493 ${riser_height}" />
+        </geometry>
+      </collision>
+    </link>
+    <joint name="riser_link_joint" type="fixed">
+      <origin xyz="0 0 ${0.225 - deck_thickness}" rpy="0 0 0" />
+      <parent link="chassis_link" />
+      <child link="riser_link" />
+    </joint>
+    <joint name="right_side_cover_link_joint" type="fixed">
+      <origin xyz="0 0 0" rpy="0 0 0" />
+      <parent link="chassis_link"/>
+      <child link="right_side_cover_link" />
+    </joint>
+    <joint name="left_side_cover_link_joint" type="fixed">
+      <origin xyz="0 0 0" rpy="0 0 0" />
+      <parent link="chassis_link"/>
+      <child link="left_side_cover_link" />
+    </joint>
+    <link name="left_side_cover_link">
+      <visual>
+        <origin xyz="0 0 0" rpy="0 0 ${PI}" />
+        <geometry>
+          <mesh filename="package://ridgeback_description/meshes/side-cover.stl"/>
+        </geometry>
+        <material name="yellow" />
+      </visual>
+    </link>
+    <link name="right_side_cover_link">
+      <visual>
+        <origin xyz="0 0 0" rpy="0 0 0" />
+        <geometry>
+          <mesh filename="package://ridgeback_description/meshes/side-cover.stl"/>
+        </geometry>
+        <material name="yellow" />
+      </visual>
+    </link>
+    <joint name="front_cover_link_joint" type="fixed">
+      <origin xyz="0 0 0" rpy="0 0 0" />
+      <parent link="chassis_link"/>
+      <child link="front_cover_link" />
+    </joint>
+    <link name="front_cover_link">
+      <visual>
+        <origin xyz="0 0 0" rpy="0 0 0" />
+        <geometry>
+          <mesh filename="package://ridgeback_description/meshes/end-cover.stl" />
+        </geometry>
+        <material name="black" />
+      </visual>
+    </link>
+    <joint name="rear_cover_link_joint" type="fixed">
+      <origin xyz="0 0 0" rpy="0 0 0" />
+      <parent link="chassis_link"/>
+      <child link="rear_cover_link" />
+    </joint>
+    <link name="rear_cover_link">
+      <visual>
+        <origin xyz="0 0 0" rpy="0 0 ${PI}" />
+        <geometry>
+          <mesh filename="package://ridgeback_description/meshes/end-cover.stl" />
+        </geometry>
+        <material name="black" />
+      </visual>
+    </link>
+    <joint name="front_lights_link_joint" type="fixed">
+      <origin xyz="0 0 0" rpy="0 0 0" />
+      <parent link="chassis_link"/>
+      <child link="front_lights_link" />
+    </joint>
+    <joint name="rear_lights_link_joint" type="fixed">
+      <origin xyz="0 0 0" rpy="0 0 0" />
+      <parent link="chassis_link"/>
+      <child link="rear_lights_link" />
+    </joint>
+    <link name="front_lights_link">
+      <visual>
+        <origin xyz="0 0 0" rpy="0 0 0" />
+        <geometry>
+          <mesh filename="package://ridgeback_description/meshes/lights.stl" />
+        </geometry>
+        <material name="white" />
+      </visual>
+    </link>
+    <link name="rear_lights_link">
+      <visual>
+        <origin xyz="0 0 0" rpy="0 0 ${PI}" />
+        <geometry>
+          <mesh filename="package://ridgeback_description/meshes/lights.stl" />
+        </geometry>
+        <material name="black" />
+      </visual>
+    </link>
+    <joint name="top_link_joint" type="fixed">
+      <origin xyz="0 0 ${riser_height-deck_height+deck_thickness}" rpy="0 0 0" />
+      <parent link="riser_link"/>
+      <child link="top_link" />
+    </joint>
+    <link name="top_link">
+      <visual>
+        <origin xyz="0 0 0" rpy="0 0 0" />
+        <geometry>
+          <mesh filename="package://ridgeback_description/meshes/top.stl" />
+        </geometry>
+        <material name="black" />
+      </visual>
+      <collision>
+        <origin xyz="0 0 0" rpy="0 0 0" />
+        <geometry>
+          <mesh filename="package://ridgeback_description/meshes/top.stl"/>
+        </geometry>
+      </collision>
+    </link>
+    <joint name="axle_joint" type="fixed">
+      <origin xyz="0 0 ${axle_offset}" rpy="0 0 0" />
+      <parent link="chassis_link"/>
+      <child link="axle_link" />
+    </joint>
+    <link name="axle_link">
+      <visual>
+        <origin xyz="0 0 0" rpy="0 ${PI/2} 0" />
+        <geometry>
+          <mesh filename="package://ridgeback_description/meshes/axle.stl" />
+        </geometry>
+        <material name="black" />
+      </visual>
+    </link>
+    <link name="imu_link">
+      <inertial>
+        <mass value="0.001"/>
+        <origin xyz="0 0 0" rpy="0 0 0"/>
+        <inertia ixx="${dummy_inertia}" ixy="0.0" ixz="0.0" iyy="${dummy_inertia}" iyz="0.0" izz="${dummy_inertia}"/>
+      </inertial>
+    </link>
+    <joint name="imu_joint" type="fixed">
+      <parent link="chassis_link" />
+      <child link="imu_link" />
+      <origin xyz="${imu_offset_x} ${imu_offset_y} ${imu_offset_z}" rpy="0 0 0"/>
+    </joint>
+    <link name="mid_mount" />
+    <joint name="mid_mount_joint" type="fixed">
+      <parent link="riser_link" />
+      <child link="mid_mount" />
+      <origin xyz="0 0 ${riser_height + deck_thickness}" rpy="0 0 0"/>
+    </joint>
   </xacro:macro>
-  <xacro:rocker prefix="front" joint_type="revolute" location="1" >
-    <limit lower="-0.08726" upper="0.08726" effort="0" velocity="0" />
-  </xacro:rocker>
-  <xacro:rocker prefix="rear" joint_type="fixed" location="-1" >
-    <limit effort="0" velocity="0" />
-  </xacro:rocker>
-  <link name="base_link"></link>
-  <joint name="base_link_joint" type="fixed">
-    <origin xyz="0 0 0" rpy="0 0 0" />
-    <parent link="base_link"/>
-    <child link="chassis_link" />
-  </joint>
-  <link name="chassis_link">
-    <visual>
-      <origin xyz="0 0 0" rpy="0 0 0" />
-      <geometry>
-        <mesh filename="package://ridgeback_description/meshes/body.stl"/>
-      </geometry>
-      <material name="black" />
-    </visual>
-    <collision>
-      <origin xyz="0 0 0"/>
-      <geometry>
-        <mesh filename="package://ridgeback_description/meshes/body-collision.stl"/>
-      </geometry>
-    </collision>
-    <inertial>
-      <origin xyz="0.012 0.002 0.067" rpy="${PI/2} 0 ${PI/2}"/>
-      <mass value="165.304"/>
-      <inertia
-        ixx="4.4744" ixy="0.03098" ixz="0.003647"
-        iyy="7.1624" iyz="0.1228"
-        izz="4.6155"/>
-    </inertial>
-  </link>
-  <link name="riser_link">
-    <visual>
-      <origin xyz="0 0 ${riser_height/2}" rpy="0 0 ${pi/4}" />
-      <geometry>
-        <box size="0.493 0.493 ${riser_height}" />
-      </geometry>
-      <material name="light_grey" />
-    </visual>
-    <collision>
-      <origin xyz="0 0 ${riser_height/2}" rpy="0 0 ${pi/4}" />
-      <geometry>
-        <box size="0.493 0.493 ${riser_height}" />
-      </geometry>
-    </collision>
-  </link>
-  <joint name="riser_link_joint" type="fixed">
-    <origin xyz="0 0 ${0.225 - deck_thickness}" rpy="0 0 0" />
-    <parent link="chassis_link" />
-    <child link="riser_link" />
-  </joint>
-  <joint name="right_side_cover_link_joint" type="fixed">
-    <origin xyz="0 0 0" rpy="0 0 0" />
-    <parent link="chassis_link"/>
-    <child link="right_side_cover_link" />
-  </joint>
-  <joint name="left_side_cover_link_joint" type="fixed">
-    <origin xyz="0 0 0" rpy="0 0 0" />
-    <parent link="chassis_link"/>
-    <child link="left_side_cover_link" />
-  </joint>
-  <link name="left_side_cover_link">
-    <visual>
-      <origin xyz="0 0 0" rpy="0 0 ${PI}" />
-      <geometry>
-        <mesh filename="package://ridgeback_description/meshes/side-cover.stl"/>
-      </geometry>
-      <material name="yellow" />
-    </visual>
-  </link>
-  <link name="right_side_cover_link">
-    <visual>
-      <origin xyz="0 0 0" rpy="0 0 0" />
-      <geometry>
-        <mesh filename="package://ridgeback_description/meshes/side-cover.stl"/>
-      </geometry>
-      <material name="yellow" />
-    </visual>
-  </link>
-  <joint name="front_cover_link_joint" type="fixed">
-    <origin xyz="0 0 0" rpy="0 0 0" />
-    <parent link="chassis_link"/>
-    <child link="front_cover_link" />
-  </joint>
-  <link name="front_cover_link">
-    <visual>
-      <origin xyz="0 0 0" rpy="0 0 0" />
-      <geometry>
-        <mesh filename="package://ridgeback_description/meshes/end-cover.stl" />
-      </geometry>
-      <material name="black" />
-    </visual>
-  </link>
-  <joint name="rear_cover_link_joint" type="fixed">
-    <origin xyz="0 0 0" rpy="0 0 0" />
-    <parent link="chassis_link"/>
-    <child link="rear_cover_link" />
-  </joint>
-  <link name="rear_cover_link">
-    <visual>
-      <origin xyz="0 0 0" rpy="0 0 ${PI}" />
-      <geometry>
-        <mesh filename="package://ridgeback_description/meshes/end-cover.stl" />
-      </geometry>
-      <material name="black" />
-    </visual>
-  </link>
-  <joint name="front_lights_link_joint" type="fixed">
-    <origin xyz="0 0 0" rpy="0 0 0" />
-    <parent link="chassis_link"/>
-    <child link="front_lights_link" />
-  </joint>
-  <joint name="rear_lights_link_joint" type="fixed">
-    <origin xyz="0 0 0" rpy="0 0 0" />
-    <parent link="chassis_link"/>
-    <child link="rear_lights_link" />
-  </joint>
-  <link name="front_lights_link">
-    <visual>
-      <origin xyz="0 0 0" rpy="0 0 0" />
-      <geometry>
-        <mesh filename="package://ridgeback_description/meshes/lights.stl" />
-      </geometry>
-      <material name="white" />
-    </visual>
-  </link>
-  <link name="rear_lights_link">
-    <visual>
-      <origin xyz="0 0 0" rpy="0 0 ${PI}" />
-      <geometry>
-        <mesh filename="package://ridgeback_description/meshes/lights.stl" />
-      </geometry>
-      <material name="black" />
-    </visual>
-  </link>
-  <joint name="top_link_joint" type="fixed">
-    <origin xyz="0 0 ${riser_height-deck_height+deck_thickness}" rpy="0 0 0" />
-    <parent link="riser_link"/>
-    <child link="top_link" />
-  </joint>
-  <link name="top_link">
-    <visual>
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
Commit message: Add parent link

File: ridgeback_description/urdf/ridgeback.urdf.xacro (robot description, xacro)
@@ -63,5 +63,5 @@
     </transmission>
   </xacro:macro>
-  <xacro:macro name="ridgeback">
+  <xacro:macro name="ridgeback" params="parent">
     <xacro:macro name="rocker" params="prefix joint_type location *joint_limits">
       <link name="${prefix}_rocker_link">
@@ -102,7 +102,8 @@
       <limit effort="0" velocity="0" />
     </xacro:rocker>
+    <link name="${parent}"/>
     <joint name="base_link_joint" type="fixed">
       <origin xyz="0 0 0" rpy="0 0 0" />
-      <parent link="base_link"/>
+      <parent link="${parent}"/>
       <child link="chassis_link" />
     </joint>
